Commit message: [Demo] Updated hardware for demo
Signed-off-by: Sergio A. Mart <sergio@earthrover.cc>

File: earth_rover_description/urdf/earth_rover.urdf.xacro (robot description, xacro)
@@ -64,4 +64,6 @@
 		<origin xyz="${base_x/2} 0 0" />
 	</joint>
+    <xacro:include filename="$(find earth_rover_description)/urdf/imu.xacro"/>
+    <xacro:include filename="$(find earth_rover_description)/urdf/gps.xacro"/>
 	<!-- gazebo tags -->
 	<gazebo>

File: earth_rover_description/urdf/imu.xacro (robot description, xacro)
@@ -9,8 +9,8 @@
   <joint name="imu_joint" type="fixed">
     <parent link="base_link"/>
-    <child link="imu"/>
+    <child link="imu_bosch_link"/>
   </joint>
  <!-- Base Link -->
-  <link name="imu">
+  <link name="imu_bosch_link">
     <collision>
       <origin xyz="0 0 0.05" rpy="0 0 0"/>
@@ -35,5 +35,5 @@
     </inertial>
   </link>
- <gazebo reference="imu">
+ <gazebo reference="imu_bosch_link">
     <material>Gazebo/Orange</material>
   </gazebo>
