Commit message: new urdf sensor file

File: simulation/sensor_sim_gazebo/urdf/sensor.xacro (robot description, xacro)
@@ -1,10 +1,8 @@
 <?xml version="1.0"?>
 <robot name="sensor" xmlns:xacro="http://www.ros.org/wiki/xacro">
-  <xacro:property name="height1" value="0.2" />
-  <xacro:property name="width" value="0.2" />
- <!-- Used for fixing robot to Gazebo 'base_link' -->
-  <link name="world"/>
-  <joint name="fixed" type="fixed">
-    <parent link="world"/>
+  <xacro:property name="height1" value="0.05" />
+  <xacro:property name="width" value="0.05" />
+   <joint name="fixed" type="fixed">
+    <parent link="battery_block_link"/>
     <child link="sensor"/>
   </joint>
